Commit message: V3 without differential

File: urdf/ERC22_URDF.xacro (robot description, xacro)
@@ -6,7 +6,7 @@
 <link name="base_link">
   <inertial>
-    <origin xyz="-0.12399606900784002 -0.9004631487269288 0.19317312158653174" rpy="0 0 0"/>
-    <mass value="1.095143414214452"/>
-    <inertia ixx="0.056886" iyy="0.063322" izz="0.105522" ixy="0.0" iyz="2e-06" ixz="0.00064"/>
+    <origin xyz="0.009257442272988727 0.0008928693179032305 0.4506338283968874" rpy="0 0 0"/>
+    <mass value="1.7296802386297885"/>
+    <inertia ixx="0.122562" iyy="0.09308" izz="0.197435" ixy="7.2e-05" iyz="0.000587" ixz="0.006199"/>
   </inertial>
   <visual>
@@ -24,112 +24,12 @@
   </collision>
 </link>
-<link name="RB_bar_1">
-  <inertial>
-    <origin xyz="-0.00043476378514936687 2.9871340390119627e-07 0.03500006530461092" rpy="0 0 0"/>
-    <mass value="0.08134271687498153"/>
-    <inertia ixx="0.002209" iyy="9e-06" izz="0.002216" ixy="0.0" iyz="0.0" ixz="0.0"/>
-  </inertial>
-  <visual>
-    <origin xyz="0.219279 0.900465 -0.267045" rpy="0 0 0"/>
-    <geometry>
-      <mesh filename="package://ERC22_URDF_description/meshes/RB_bar_1.stl" scale="0.001 0.001 0.001"/>
-    </geometry>
-    <material name="silver"/>
-  </visual>
-  <collision>
-    <origin xyz="0.219279 0.900465 -0.267045" rpy="0 0 0"/>
-    <geometry>
-      <mesh filename="package://ERC22_URDF_description/meshes/RB_bar_1.stl" scale="0.001 0.001 0.001"/>
-    </geometry>
-  </collision>
-</link>
-<link name="Rocker_bogie_union_v1_1">
-  <inertial>
-    <origin xyz="0.057709013481098526 -0.00048140313745825836 -0.00983122565203498" rpy="0 0 0"/>
-    <mass value="0.0012126519563795419"/>
-    <inertia ixx="0.0" iyy="2e-06" izz="2e-06" ixy="0.0" iyz="-0.0" ixz="0.0"/>
-  </inertial>
-  <visual>
-    <origin xyz="0.219246 1.185465 -0.307045" rpy="0 0 0"/>
-    <geometry>
-      <mesh filename="package://ERC22_URDF_description/meshes/Rocker_bogie_union_v1_1.stl" scale="0.001 0.001 0.001"/>
-    </geometry>
-    <material name="silver"/>
-  </visual>
-  <collision>
-    <origin xyz="0.219246 1.185465 -0.307045" rpy="0 0 0"/>
-    <geometry>
-      <mesh filename="package://ERC22_URDF_description/meshes/Rocker_bogie_union_v1_1.stl" scale="0.001 0.001 0.001"/>
-    </geometry>
-  </collision>
-</link>
-<link name="Left_leg_single_1">
-  <inertial>
-    <origin xyz="0.366932298339489 -0.5890477556142102 0.9361370079778285" rpy="0 0 0"/>
-    <mass value="0.2886052811001981"/>
-    <inertia ixx="0.00105" iyy="0.01212" izz="0.011639" ixy="0.001022" iyz="-0.000342" ixz="0.002262"/>
-  </inertial>
-  <visual>
-    <origin xyz="0.373006 0.635095 0.768259" rpy="0 0 0"/>
-    <geometry>
-      <mesh filename="package://ERC22_URDF_description/meshes/Left_leg_single_1.stl" scale="0.001 0.001 0.001"/>
-    </geometry>
-    <material name="silver"/>
-  </visual>
-  <collision>
-    <origin xyz="0.373006 0.635095 0.768259" rpy="0 0 0"/>
-    <geometry>
-      <mesh filename="package://ERC22_URDF_description/meshes/Left_leg_single_1.stl" scale="0.001 0.001 0.001"/>
-    </geometry>
-  </collision>
-</link>
-<link name="Left_axis_1">
-  <inertial>
-    <origin xyz="4.276494046384638e-08 -0.035617360363259465 4.507138290102408e-05" rpy="0 0 0"/>
-    <mass value="0.02866313110747046"/>
-    <inertia ixx="2.1e-05" iyy="1e-06" izz="2.1e-05" ixy="-0.0" iyz="-0.0" ixz="0.0"/>
-  </inertial>
-  <visual>
-    <origin xyz="0.100777 1.150462 -0.187044" rpy="0 0 0"/>
-    <geometry>
-      <mesh filename="package://ERC22_URDF_description/meshes/Left_axis_1.stl" scale="0.001 0.001 0.001"/>
-    </geometry>
-    <material name="silver"/>
-  </visual>
-  <collision>
-    <origin xyz="0.100777 1.150462 -0.187044" rpy="0 0 0"/>
-    <geometry>
-      <mesh filename="package://ERC22_URDF_description/meshes/Left_axis_1.stl" scale="0.001 0.001 0.001"/>
-    </geometry>
-  </collision>
-</link>
-<link name="Left_leg_single_1">
-  <inertial>
-    <origin xyz="0.09470329833948897 -0.06368075561421005 -0.019165992022171507" rpy="0 0 0"/>
-    <mass value="0.2886052811001981"/>
-    <inertia ixx="0.00105" iyy="0.01212" izz="0.011639" ixy="0.001022" iyz="-0.000342" ixz="0.002262"/>
-  </inertial>
-  <visual>
-    <origin xyz="0.100777 1.160462 -0.187044" rpy="0 0 0"/>
-    <geometry>
-      <mesh filename="package://ERC22_URDF_description/meshes/Left_leg_single_1.stl" scale="0.001 0.001 0.001"/>
-    </geometry>
-    <material name="silver"/>
-  </visual>
-  <collision>
-    <origin xyz="0.100777 1.160462 -0.187044" rpy="0 0 0"/>
-    <geometry>
-      <mesh filename="package://ERC22_URDF_description/meshes/Left_leg_single_1.stl" scale="0.001 0.001 0.001"/>
-    </geometry>
-  </collision>
-</link>
 <link name="WLF_supp_1">
   <inertial>
-    <origin xyz="-0.001281629539594098 0.044567971064483736 -0.07032194715949266" rpy="0 0 0"/>
-    <mass value="0.040963204487274314"/>
-    <inertia ixx="0.000114" iyy="9.6e-05" izz="3e-05" ixy="0.0" iyz="1.6e-05" ixz="-2e-06"/>
-  </inertial>
-  <visual>
-    <origin xyz="-0.297237 1.288962 -0.08655" rpy="0 0 0"/>
+    <origin xyz="0.0010155899598203177 0.04456811672884159 -0.069974852362928" rpy="0 0 0"/>
+    <mass value="0.040963207008450755"/>
+    <inertia ixx="0.000114" iyy="9.6e-05" izz="3e-05" ixy="-0.0" iyz="1.6e-05" ixz="1e-06"/>
+  </inertial>
+  <visual>
+    <origin xyz="-0.393441 0.383158 -0.365642" rpy="0 0 0"/>
     <geometry>
       <mesh filename="package://ERC22_URDF_description/meshes/WLF_supp_1.stl" scale="0.001 0.001 0.001"/>
@@ -138,5 +38,5 @@
   </visual>
   <collision>
-    <origin xyz="-0.297237 1.288962 -0.08655" rpy="0 0 0"/>
+    <origin xyz="-0.393441 0.383158 -0.365642" rpy="0 0 0"/>
     <geometry>
       <mesh filename="package://ERC22_URDF_description/meshes/WLF_supp_1.stl" scale="0.001 0.001 0.001"/>
@@ -144,12 +44,92 @@
   </collision>
 </link>
+<link name="Left_leg_double_1">
+  <inertial>
+    <origin xyz="-0.022088532350106327 -0.06278452284012143 -0.07367590613643721" rpy="0 0 0"/>
+    <mass value="0.1583068780205665"/>
+    <inertia ixx="0.000845" iyy="0.003257" izz="0.002543" ixy="-0.000166" iyz="-2.5e-05" ixz="0.000841"/>
+  </inertial>
+  <visual>
+    <origin xyz="0.25259 0.310658 -0.447478" rpy="0 0 0"/>
+    <geometry>
+      <mesh filename="package://ERC22_URDF_description/meshes/Left_leg_double_1.stl" scale="0.001 0.001 0.001"/>
+    </geometry>
+    <material name="silver"/>
+  </visual>
+  <collision>
+    <origin xyz="0.25259 0.310658 -0.447478" rpy="0 0 0"/>
+    <geometry>
+      <mesh filename="package://ERC22_URDF_description/meshes/Left_leg_double_1.stl" scale="0.001 0.001 0.001"/>
+    </geometry>
+  </collision>
+</link>
+<link name="WLB_supp_1">
+  <inertial>
+    <origin xyz="-0.0028618909710108054 0.03188196836487278 -0.06602065383277494" rpy="0 0 0"/>
+    <mass value="0.05726725763420208"/>
+    <inertia ixx="0.000209" iyy="0.000168" izz="5.9e-05" ixy="2e-06" iyz="5.6e-05" ixz="-7e-06"/>
+  </inertial>
+  <visual>
+    <origin xyz="0.432452 0.392158 -0.376754" rpy="0 0 0"/>
+    <geometry>
+      <mesh filename="package://ERC22_URDF_description/meshes/WLB_supp_1.stl" scale="0.001 0.001 0.001"/>
+    </geometry>
+    <material name="silver"/>
+  </visual>
+  <collision>
+    <origin xyz="0.432452 0.392158 -0.376754" rpy="0 0 0"/>
+    <geometry>
+      <mesh filename="package://ERC22_URDF_description/meshes/WLB_supp_1.stl" scale="0.001 0.001 0.001"/>
+    </geometry>
+  </collision>
+</link>
+<link name="WLB_1">
+  <inertial>
+    <origin xyz="-0.00015756056275473274 -0.048534670780080114 6.7474958049262845e-06" rpy="0 0 0"/>
+    <mass value="0.821177966951147"/>
+    <inertia ixx="0.002537" iyy="0.004162" izz="0.002536" ixy="6e-06" iyz="-0.0" ixz="0.0"/>
+  </inertial>
+  <visual>
+    <origin xyz="0.439051 0.373675 -0.218892" rpy="0 0 0"/>
+    <geometry>
+      <mesh filename="package://ERC22_URDF_description/meshes/WLB_1.stl" scale="0.001 0.001 0.001"/>
+    </geometry>
+    <material name="silver"/>
+  </visual>
+  <collision>
+    <origin xyz="0.439051 0.373675 -0.218892" rpy="0 0 0"/>
+    <geometry>
+      <mesh filename="package://ERC22_URDF_description/meshes/WLB_1.stl" scale="0.001 0.001 0.001"/>
+    </geometry>
+  </collision>
+</link>
+<link name="WLM_1">
+  <inertial>
+    <origin xyz="-4.7183024518004935e-07 -0.05483339443238905 8.441033064188197e-08" rpy="0 0 0"/>
+    <mass value="0.8017382692848779"/>
+    <inertia ixx="0.002476" iyy="0.004159" izz="0.002476" ixy="0.0" iyz="0.0" ixz="0.0"/>
+  </inertial>
+  <visual>
+    <origin xyz="0.039463 0.380158 -0.191263" rpy="0 0 0"/>
+    <geometry>
+      <mesh filename="package://ERC22_URDF_description/meshes/WLM_1.stl" scale="0.001 0.001 0.001"/>
+    </geometry>
+    <material name="silver"/>
+  </visual>
+  <collision>
+    <origin xyz="0.039463 0.380158 -0.191263" rpy="0 0 0"/>
+    <geometry>
+      <mesh filename="package://ERC22_URDF_description/meshes/WLM_1.stl" scale="0.001 0.001 0.001"/>
+    </geometry>
+  </collision>
+</link>
 <link name="WLF_1">
   <inertial>
-    <origin xyz="0.00029170484983265244 -0.04048463060522245 -2.796167765266311e-06" rpy="0 0 0"/>
-    <mass value="0.7923139934667868"/>
-    <inertia ixx="0.002447" iyy="0.004158" izz="0.002446" ixy="-1.2e-05" iyz="0.0" ixz="-0.0"/>
-  </inertial>
-  <visual>
-    <origin xyz="-0.295688 1.270479 0.053793" rpy="0 0 0"/>
+    <origin xyz="0.00034773001940091586 -0.048246876176874454 7.974817149869473e-06" rpy="0 0 0"/>
+    <mass value="0.8211285553800025"/>
+    <inertia ixx="0.002536" iyy="0.004162" izz="0.002535" ixy="-1.2e-05" iyz="-0.0" ixz="-0.0"/>
+  </inertial>
+  <visual>
+    <origin xyz="-0.396484 0.364675 -0.225675" rpy="0 0 0"/>
     <geometry>
       <mesh filename="package://ERC22_URDF_description/meshes/WLF_1.stl" scale="0.001 0.001 0.001"/>
@@ -158,5 +138,5 @@
   </visual>
   <collision>
-    <origin xyz="-0.295688 1.270479 0.053793" rpy="0 0 0"/>
+    <origin xyz="-0.396484 0.364675 -0.225675" rpy="0 0 0"/>
     <geometry>
       <mesh filename="package://ERC22_URDF_description/meshes/WLF_1.stl" scale="0.001 0.001 0.001"/>
@@ -164,201 +144,101 @@
   </collision>
 </link>
-<link name="Left_axis_SD_1">
-  <inertial>
-    <origin xyz="1.5367052003112391e-07 -0.03475915283616948 1.0535873512518279e-07" rpy="0 0 0"/>
-    <mass value="0.025317599264113037"/>
-    <inertia ixx="1.3e-05" iyy="3e-06" izz="1.3e-05" ixy="-0.0" iyz="-0.0" ixz="0.0"/>
-  </inertial>
-  <visual>
-    <origin xyz="0.345765 1.216462 -0.189514" rpy="0 0 0"/>
-    <geometry>
-      <mesh filename="package://ERC22_URDF_description/meshes/Left_axis_SD_1.stl" scale="0.001 0.001 0.001"/>
-    </geometry>
-    <material name="silver"/>
-  </visual>
-  <collision>
-    <origin xyz="0.345765 1.216462 -0.189514" rpy="0 0 0"/>
-    <geometry>
-      <mesh filename="package://ERC22_URDF_description/meshes/Left_axis_SD_1.stl" scale="0.001 0.001 0.001"/>
-    </geometry>
-  </collision>
-</link>
-<link name="Left_leg_double_1">
-  <inertial>
-    <origin xyz="-0.024102248154190542 -0.01780597583428034 -0.0880459072969701" rpy="0 0 0"/>
-    <mass value="0.1333867080829175"/>
-    <inertia ixx="0.000613" iyy="0.00308" izz="0.00254" ixy="-0.00015" iyz="2.4e-05" ixz="0.000844"/>
-  </inertial>
-  <visual>
-    <origin xyz="0.345765 1.262462 -0.189514" rpy="0 0 0"/>
-    <geometry>
-      <mesh filename="package://ERC22_URDF_description/meshes/Left_leg_double_1.stl" scale="0.001 0.001 0.001"/>
-    </geometry>
-    <material name="silver"/>
-  </visual>
-  <collision>
-    <origin xyz="0.345765 1.262462 -0.189514" rpy="0 0 0"/>
-    <geometry>
-      <mesh filename="package://ERC22_URDF_description/meshes/Left_leg_double_1.stl" scale="0.001 0.001 0.001"/>
-    </geometry>
-  </collision>
-</link>
-<link name="WLB_supp_1">
-  <inertial>
-    <origin xyz="-0.0013739737228875004 0.03188140888878954 -0.06606839757279151" rpy="0 0 0"/>
-    <mass value="0.05726725752231377"/>
-    <inertia ixx="0.000209" iyy="0.000168" izz="5.9e-05" ixy="1e-06" iyz="5.6e-05" ixz="-4e-06"/>
-  </inertial>
-  <visual>
-    <origin xyz="0.523872 1.294462 -0.11448" rpy="0 0 0"/>
-    <geometry>
-      <mesh filename="package://ERC22_URDF_description/meshes/WLB_supp_1.stl" scale="0.001 0.001 0.001"/>
-    </geometry>
-    <material name="silver"/>
-  </visual>
-  <collision>
-    <origin xyz="0.523872 1.294462 -0.11448" rpy="0 0 0"/>
-    <geometry>
-      <mesh filename="package://ERC22_URDF_description/meshes/WLB_supp_1.stl" scale="0.001 0.001 0.001"/>
-    </geometry>
-  </collision>
-</link>
-<link name="WLB_1">
-  <inertial>
-    <origin xyz="-6.916339846396724e-07 -0.040485221549373174 5.47043015268478e-07" rpy="0 0 0"/>
-    <mass value="0.7923134916389618"/>
-    <inertia ixx="0.002446" iyy="0.004158" izz="0.002446" ixy="0.0" iyz="0.0" ixz="0.0"/>
-  </inertial>
-  <visual>
-    <origin xyz="0.526728 1.275979 0.043494" rpy="0 0 0"/>
-    <geometry>
-      <mesh filename="package://ERC22_URDF_description/meshes/WLB_1.stl" scale="0.001 0.001 0.001"/>
-    </geometry>
-    <material name="silver"/>
-  </visual>
-  <collision>
-    <origin xyz="0.526728 1.275979 0.043494" rpy="0 0 0"/>
-    <geometry>
-      <mesh filename="package://ERC22_URDF_description/meshes/WLB_1.stl" scale="0.001 0.001 0.001"/>
-    </geometry>
-  </collision>
-</link>
-<link name="WLM_1">
-  <inertial>
-    <origin xyz="-6.161896191625438e-07 -0.04048579284392173 -7.482984916359903e-07" rpy="0 0 0"/>
-    <mass value="0.7923134916400008"/>
-    <inertia ixx="0.002446" iyy="0.004158" izz="0.002446" ixy="-0.0" iyz="0.0" ixz="-0.0"/>
-  </inertial>
-  <visual>
-    <origin xyz="0.12653 1.282462 0.061494" rpy="0 0 0"/>
-    <geometry>
-      <mesh filename="package://ERC22_URDF_description/meshes/WLM_1.stl" scale="0.001 0.001 0.001"/>
-    </geometry>
-    <material name="silver"/>
-  </visual>
-  <collision>
-    <origin xyz="0.12653 1.282462 0.061494" rpy="0 0 0"/>
-    <geometry>
-      <mesh filename="package://ERC22_URDF_description/meshes/WLM_1.stl" scale="0.001 0.001 0.001"/>
-    </geometry>
-  </collision>
-</link>
-<link name="Rocker_bogie_union_v1_2">
-  <inertial>
-    <origin xyz="0.05770920163164456 0.0004837912765092156 -0.009830910675701965" rpy="0 0 0"/>
-    <mass value="0.0012126519563795419"/>
-    <inertia ixx="0.0" iyy="2e-06" izz="2e-06" ixy="-0.0" iyz="0.0" ixz="0.0"/>
-  </inertial>
-  <visual>
-    <origin xyz="0.219313 0.615465 -0.307045" rpy="0 0 0"/>
-    <geometry>
-      <mesh filename="package://ERC22_URDF_description/meshes/Rocker_bogie_union_v1_2.stl" scale="0.001 0.001 0.001"/>
-    </geometry>
-    <material name="silver"/>
-  </visual>
-  <collision>
-    <origin xyz="0.219313 0.615465 -0.307045" rpy="0 0 0"/>
-    <geometry>
-      <mesh filename="package://ERC22_URDF_description/meshes/Rocker_bogie_union_v1_2.stl" scale="0.001 0.001 0.001"/>
-    </geometry>
-  </collision>
-</link>
-<link name="Right_axis_1">
-  <inertial>
-    <origin xyz="4.276494013077947e-08 0.035882771227694454 4.507138290132939e-05" rpy="0 0 0"/>
-    <mass value="0.028663131107470416"/>
-    <inertia ixx="2.1e-05" iyy="1e-06" izz="2.1e-05" ixy="-0.0" iyz="-0.0" ixz="-0.0"/>
-  </inertial>
-  <visual>
-    <origin xyz="0.100777 0.650463 -0.187044" rpy="0 0 0"/>
-    <geometry>
-      <mesh filename="package://ERC22_URDF_description/meshes/Right_axis_1.stl" scale="0.001 0.001 0.001"/>
-    </geometry>
-    <material name="silver"/>
-  </visual>
-  <collision>
-    <origin xyz="0.100777 0.650463 -0.187044" rpy="0 0 0"/>
-    <geometry>
-      <mesh filename="package://ERC22_URDF_description/meshes/Right_axis_1.stl" scale="0.001 0.001 0.001"/>
-    </geometry>
-  </collision>
-</link>
-<link name="Right_leg_single_1">
-  <inertial>
-    <origin xyz="0.09365647258574741 0.6096789528898845 -0.12409973710729968" rpy="0 0 0"/>
-    <mass value="0.2886052811002028"/>
-    <inertia ixx="0.001047" iyy="0.01212" izz="0.011642" ixy="-0.001022" iyz="0.000341" ixz="0.002255"/>
-  </inertial>
-  <visual>
-    <origin xyz="0.099718 1.186462 -0.292038" rpy="0 0 0"/>
-    <geometry>
-      <mesh filename="package://ERC22_URDF_description/meshes/Right_leg_single_1.stl" scale="0.001 0.001 0.001"/>
-    </geometry>
-    <material name="silver"/>
-  </visual>
-  <collision>
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