Commit message: Joints name more descriptive

File: urdf/ERC22_URDF.xacro (robot description, xacro)
@@ -6,7 +6,7 @@
 <link name="base_link">
   <inertial>
-    <origin xyz="0.009439051177251773 0.0008928693179034862 0.4515443268163816" rpy="0 0 0"/>
-    <mass value="1.7296802386297903"/>
-    <inertia ixx="0.122252" iyy="0.093075" izz="0.197741" ixy="-4.9e-05" iyz="2.2e-05" ixz="0.005471"/>
+    <origin xyz="0.009312479330910419 0.0008928693179026247 0.4508429285266153" rpy="0 0 0"/>
+    <mass value="1.729680238629788"/>
+    <inertia ixx="0.122469" iyy="0.093078" izz="0.197526" ixy="-5.1e-05" iyz="1.2e-05" ixz="0.006038"/>
   </inertial>
   <visual>
@@ -26,10 +26,10 @@
 <link name="WLF_supp_1">
   <inertial>
-    <origin xyz="0.0010155899598203177 0.04456811672884159 -0.069974852362928" rpy="0 0 0"/>
+    <origin xyz="-0.0005722202916380592 0.04456811672884131 -0.06998013314667545" rpy="0 0 0"/>
     <mass value="0.040963207008450755"/>
-    <inertia ixx="0.000114" iyy="9.6e-05" izz="3e-05" ixy="-0.0" iyz="1.6e-05" ixz="1e-06"/>
-  </inertial>
-  <visual>
-    <origin xyz="-0.393441 0.383158 -0.365642" rpy="0 0 0"/>
+    <inertia ixx="0.000114" iyy="9.6e-05" izz="3e-05" ixy="-0.0" iyz="1.6e-05" ixz="-1e-06"/>
+  </inertial>
+  <visual>
+    <origin xyz="-0.391355 0.383158 -0.356565" rpy="0 0 0"/>
     <geometry>
       <mesh filename="package://ERC22_URDF_description/meshes/WLF_supp_1.stl" scale="0.001 0.001 0.001"/>
@@ -38,5 +38,5 @@
   </visual>
   <collision>
-    <origin xyz="-0.393441 0.383158 -0.365642" rpy="0 0 0"/>
+    <origin xyz="-0.391355 0.383158 -0.356565" rpy="0 0 0"/>
     <geometry>
       <mesh filename="package://ERC22_URDF_description/meshes/WLF_supp_1.stl" scale="0.001 0.001 0.001"/>
@@ -46,10 +46,10 @@
 <link name="Left_leg_double_1">
   <inertial>
-    <origin xyz="-0.015583210905782074 -0.06278452280466362 -0.07532072866040473" rpy="0 0 0"/>
-    <mass value="0.15830687785841724"/>
-    <inertia ixx="0.000712" iyy="0.003257" izz="0.002676" ixy="-0.000163" iyz="-3.9e-05" ixz="0.000681"/>
-  </inertial>
-  <visual>
-    <origin xyz="0.25259 0.310658 -0.447478" rpy="0 0 0"/>
+    <origin xyz="-0.017610729784847123 -0.06278452284012215 -0.07487224121996011" rpy="0 0 0"/>
+    <mass value="0.1583068780205665"/>
+    <inertia ixx="0.00075" iyy="0.003257" izz="0.002638" ixy="-0.000164" iyz="-3.5e-05" ixz="0.000733"/>
+  </inertial>
+  <visual>
+    <origin xyz="0.252653 0.310658 -0.453036" rpy="0 0 0"/>
     <geometry>
       <mesh filename="package://ERC22_URDF_description/meshes/Left_leg_double_1.stl" scale="0.001 0.001 0.001"/>
@@ -58,5 +58,5 @@
   </visual>
   <collision>
-    <origin xyz="0.25259 0.310658 -0.447478" rpy="0 0 0"/>
+    <origin xyz="0.252653 0.310658 -0.453036" rpy="0 0 0"/>
     <geometry>
       <mesh filename="package://ERC22_URDF_description/meshes/Left_leg_double_1.stl" scale="0.001 0.001 0.001"/>
@@ -66,10 +66,10 @@
 <link name="WLB_supp_1">
   <inertial>
-    <origin xyz="0.002903499921163455 0.03188196836487295 -0.06601877471300915" rpy="0 0 0"/>
+    <origin xyz="0.0011204573839502796 0.031881968364872504 -0.06607317272822505" rpy="0 0 0"/>
     <mass value="0.05726725763420208"/>
-    <inertia ixx="0.000209" iyy="0.000168" izz="5.9e-05" ixy="-3e-06" iyz="5.6e-05" ixz="6e-06"/>
-  </inertial>
-  <visual>
-    <origin xyz="0.425604 0.392158 -0.361347" rpy="0 0 0"/>
+    <inertia ixx="0.000209" iyy="0.000168" izz="5.9e-05" ixy="-1e-06" iyz="5.6e-05" ixz="2e-06"/>
+  </inertial>
+  <visual>
+    <origin xyz="0.427929 0.392158 -0.371607" rpy="0 0 0"/>
     <geometry>
       <mesh filename="package://ERC22_URDF_description/meshes/WLB_supp_1.stl" scale="0.001 0.001 0.001"/>
@@ -78,5 +78,5 @@
   </visual>
   <collision>
-    <origin xyz="0.425604 0.392158 -0.361347" rpy="0 0 0"/>
+    <origin xyz="0.427929 0.392158 -0.371607" rpy="0 0 0"/>
     <geometry>
       <mesh filename="package://ERC22_URDF_description/meshes/WLB_supp_1.stl" scale="0.001 0.001 0.001"/>
@@ -86,10 +86,10 @@
 <link name="WLB_1">
   <inertial>
-    <origin xyz="-0.000157436619810436 -0.04853467078007917 -7.357831886489752e-06" rpy="0 0 0"/>
+    <origin xyz="-0.000157582105088927 -0.04853467078008089 -2.617517294800642e-06" rpy="0 0 0"/>
     <mass value="0.821177966951147"/>
     <inertia ixx="0.002537" iyy="0.004162" izz="0.002536" ixy="6e-06" iyz="0.0" ixz="0.0"/>
   </inertial>
   <visual>
-    <origin xyz="0.418419 0.373675 -0.203511" rpy="0 0 0"/>
+    <origin xyz="0.425007 0.373675 -0.213634" rpy="0 0 0"/>
     <geometry>
       <mesh filename="package://ERC22_URDF_description/meshes/WLB_1.stl" scale="0.001 0.001 0.001"/>
@@ -98,5 +98,5 @@
   </visual>
   <collision>
-    <origin xyz="0.418419 0.373675 -0.203511" rpy="0 0 0"/>
+    <origin xyz="0.425007 0.373675 -0.213634" rpy="0 0 0"/>
     <geometry>
       <mesh filename="package://ERC22_URDF_description/meshes/WLB_1.stl" scale="0.001 0.001 0.001"/>
@@ -106,10 +106,10 @@
 <link name="WLM_1">
   <inertial>
-    <origin xyz="-9.162353946969015e-07 -0.04483339443239004 -7.236476196326169e-07" rpy="0 0 0"/>
+    <origin xyz="-7.105685515228222e-07 -0.05483339443238944 1.1425396012620936e-07" rpy="0 0 0"/>
     <mass value="0.8017382692848779"/>
     <inertia ixx="0.002476" iyy="0.004159" izz="0.002476" ixy="0.0" iyz="0.0" ixz="0.0"/>
   </inertial>
   <visual>
-    <origin xyz="0.017943 0.380158 -0.210814" rpy="0 0 0"/>
+    <origin xyz="0.02448 0.380158 -0.210124" rpy="0 0 0"/>
     <geometry>
       <mesh filename="package://ERC22_URDF_description/meshes/WLM_1.stl" scale="0.001 0.001 0.001"/>
@@ -118,5 +118,5 @@
   </visual>
   <collision>
-    <origin xyz="0.017943 0.380158 -0.210814" rpy="0 0 0"/>
+    <origin xyz="0.02448 0.380158 -0.210124" rpy="0 0 0"/>
     <geometry>
       <mesh filename="package://ERC22_URDF_description/meshes/WLM_1.stl" scale="0.001 0.001 0.001"/>
@@ -126,10 +126,10 @@
 <link name="WLF_1">
   <inertial>
-    <origin xyz="0.0002756316511097756 -0.03824713622289272 6.33834755653373e-06" rpy="0 0 0"/>
+    <origin xyz="0.00034755415545323354 -0.04824687617687501 -1.7828776904815768e-07" rpy="0 0 0"/>
     <mass value="0.8211285553800025"/>
-    <inertia ixx="0.002536" iyy="0.004162" izz="0.002535" ixy="-1.2e-05" iyz="-0.0" ixz="-0.0"/>
-  </inertial>
-  <visual>
-    <origin xyz="-0.396484 0.364675 -0.225675" rpy="0 0 0"/>
+    <inertia ixx="0.002536" iyy="0.004162" izz="0.002535" ixy="-1.2e-05" iyz="0.0" ixz="-0.0"/>
+  </inertial>
+  <visual>
+    <origin xyz="-0.391222 0.364675 -0.216565" rpy="0 0 0"/>
     <geometry>
       <mesh filename="package://ERC22_URDF_description/meshes/WLF_1.stl" scale="0.001 0.001 0.001"/>
@@ -138,5 +138,5 @@
   </visual>
   <collision>
-    <origin xyz="-0.396484 0.364675 -0.225675" rpy="0 0 0"/>
+    <origin xyz="-0.391222 0.364675 -0.216565" rpy="0 0 0"/>
     <geometry>
       <mesh filename="package://ERC22_URDF_description/meshes/WLF_1.stl" scale="0.001 0.001 0.001"/>
@@ -146,10 +146,10 @@
 <link name="WRF_supp_1">
   <inertial>
-    <origin xyz="0.0016416095063517266 -0.037844265968987045 -0.0964909033672866" rpy="0 0 0"/>
+    <origin xyz="-0.0004356849889970982 -0.037844265968987545 -0.09650313579211883" rpy="0 0 0"/>
     <mass value="0.06594197827899752"/>
-    <inertia ixx="0.000199" iyy="0.000176" izz="3.9e-05" ixy="-0.0" iyz="3e-06" ixz="3e-06"/>
-  </inertial>
-  <visual>
-    <origin xyz="-0.393337 -0.386841 -0.36517" rpy="0 0 0"/>
+    <inertia ixx="0.000199" iyy="0.000176" izz="3.9e-05" ixy="0.0" iyz="3e-06" ixz="-0.0"/>
+  </inertial>
+  <visual>
+    <origin xyz="-0.391354 -0.386841 -0.356561" rpy="0 0 0"/>
     <geometry>
       <mesh filename="package://ERC22_URDF_description/meshes/WRF_supp_1.stl" scale="0.001 0.001 0.001"/>
@@ -158,5 +158,5 @@
   </visual>
   <collision>
-    <origin xyz="-0.393337 -0.386841 -0.36517" rpy="0 0 0"/>
+    <origin xyz="-0.391354 -0.386841 -0.356561" rpy="0 0 0"/>
     <geometry>
       <mesh filename="package://ERC22_URDF_description/meshes/WRF_supp_1.stl" scale="0.001 0.001 0.001"/>
@@ -166,10 +166,10 @@
 <link name="WRB_supp_1">
   <inertial>
-    <origin xyz="0.00278870991833563 -0.031841488157177744 -0.06644057204157627" rpy="0 0 0"/>
+    <origin xyz="0.0010379712309944722 -0.03184148815717791 -0.06649153329813762" rpy="0 0 0"/>
     <mass value="0.05751878988929576"/>
-    <inertia ixx="0.000211" iyy="0.000171" izz="5.9e-05" ixy="3e-06" iyz="-5.6e-05" ixz="6e-06"/>
-  </inertial>
-  <visual>
-    <origin xyz="0.425538 -0.396591 -0.36149" rpy="0 0 0"/>
+    <inertia ixx="0.000212" iyy="0.000171" izz="5.9e-05" ixy="1e-06" iyz="-5.6e-05" ixz="2e-06"/>
+  </inertial>
+  <visual>
+    <origin xyz="0.427806 -0.396591 -0.371346" rpy="0 0 0"/>
     <geometry>
       <mesh filename="package://ERC22_URDF_description/meshes/WRB_supp_1.stl" scale="0.001 0.001 0.001"/>
@@ -178,5 +178,5 @@
   </visual>
   <collision>
-    <origin xyz="0.425538 -0.396591 -0.36149" rpy="0 0 0"/>
+    <origin xyz="0.427806 -0.396591 -0.371346" rpy="0 0 0"/>
     <geometry>
       <mesh filename="package://ERC22_URDF_description/meshes/WRB_supp_1.stl" scale="0.001 0.001 0.001"/>
@@ -186,10 +186,10 @@
 <link name="WRF_1">
   <inertial>
-    <origin xyz="0.00022243797779680774 0.030856418914129602 5.266976624562769e-06" rpy="0 0 0"/>
+    <origin xyz="0.00022231321115867564 0.030856418914129602 6.118055645987219e-07" rpy="0 0 0"/>
     <mass value="0.7923140233383783"/>
     <inertia ixx="0.002447" iyy="0.004158" izz="0.002447" ixy="1.2e-05" iyz="0.0" ixz="-0.0"/>
   </inertial>
   <visual>
-    <origin xyz="-0.396266 -0.375303 -0.2252" rpy="0 0 0"/>
+    <origin xyz="-0.39127 -0.375303 -0.216561" rpy="0 0 0"/>
     <geometry>
       <mesh filename="package://ERC22_URDF_description/meshes/WRF_1.stl" scale="0.001 0.001 0.001"/>
@@ -198,5 +198,5 @@
   </visual>
   <collision>
-    <origin xyz="-0.396266 -0.375303 -0.2252" rpy="0 0 0"/>
+    <origin xyz="-0.39127 -0.375303 -0.216561" rpy="0 0 0"/>
     <geometry>
       <mesh filename="package://ERC22_URDF_description/meshes/WRF_1.stl" scale="0.001 0.001 0.001"/>
@@ -206,10 +206,10 @@
 <link name="WRM_1">
   <inertial>
-    <origin xyz="-4.796690451780439e-07 0.04421440445825542 -3.055120773864939e-07" rpy="0 0 0"/>
+    <origin xyz="-7.423233885535396e-07 0.04421440445825414 -8.285402313679135e-07" rpy="0 0 0"/>
     <mass value="0.8108718866431287"/>
     <inertia ixx="0.002505" iyy="0.004161" izz="0.002505" ixy="0.0" iyz="0.0" ixz="0.0"/>
   </inertial>
   <visual>
-    <origin xyz="0.017751 -0.384591 -0.211299" rpy="0 0 0"/>
+    <origin xyz="0.024115 -0.384591 -0.21047" rpy="0 0 0"/>
     <geometry>
       <mesh filename="package://ERC22_URDF_description/meshes/WRM_1.stl" scale="0.001 0.001 0.001"/>
@@ -218,5 +218,5 @@
   </visual>
   <collision>
-    <origin xyz="0.017751 -0.384591 -0.211299" rpy="0 0 0"/>
+    <origin xyz="0.024115 -0.384591 -0.21047" rpy="0 0 0"/>
     <geometry>
       <mesh filename="package://ERC22_URDF_description/meshes/WRM_1.stl" scale="0.001 0.001 0.001"/>
@@ -226,10 +226,10 @@
 <link name="WRB_1">
   <inertial>
-    <origin xyz="-1.0298475141001795e-06 0.04853448757279211 4.442527895276438e-07" rpy="0 0 0"/>
+    <origin xyz="-6.598539384894408e-07 0.04853448757279283 5.190034971513935e-07" rpy="0 0 0"/>
     <mass value="0.8211769381894314"/>
     <inertia ixx="0.002537" iyy="0.004163" izz="0.002537" ixy="0.0" iyz="0.0" ixz="0.0"/>
   </inertial>
   <visual>
-    <origin xyz="0.41828 -0.378107 -0.203657" rpy="0 0 0"/>
+    <origin xyz="0.424707 -0.378107 -0.213376" rpy="0 0 0"/>
     <geometry>
       <mesh filename="package://ERC22_URDF_description/meshes/WRB_1.stl" scale="0.001 0.001 0.001"/>
@@ -238,5 +238,5 @@
   </visual>
   <collision>
-    <origin xyz="0.41828 -0.378107 -0.203657" rpy="0 0 0"/>
+    <origin xyz="0.424707 -0.378107 -0.213376" rpy="0 0 0"/>
     <geometry>
       <mesh filename="package://ERC22_URDF_description/meshes/WRB_1.stl" scale="0.001 0.001 0.001"/>
@@ -246,10 +246,10 @@
 <link name="Right_leg_double_1">
   <inertial>
-    <origin xyz="-0.01841993942514597 0.06805532100441675 -0.08940771566700395" rpy="0 0 0"/>
-    <mass value="0.1333867163635017"/>
-    <inertia ixx="0.000513" iyy="0.00308" izz="0.00264" ixy="0.000152" iyz="-1.5e-05" ixz="0.000714"/>
-  </inertial>
-  <visual>
-    <origin xyz="0.252596 -0.314341 -0.447766" rpy="0 0 0"/>
+    <origin xyz="-0.01745444401971802 0.06338178542499118 -0.07471145682820046" rpy="0 0 0"/>
+    <mass value="0.15870353264297354"/>
+    <inertia ixx="0.000751" iyy="0.00326" izz="0.002641" ixy="0.000164" iyz="3.7e-05" ixz="0.00073"/>
+  </inertial>
+  <visual>
+    <origin xyz="0.252653 -0.314341 -0.453038" rpy="0 0 0"/>
     <geometry>
       <mesh filename="package://ERC22_URDF_description/meshes/Right_leg_double_1.stl" scale="0.001 0.001 0.001"/>
@@ -258,5 +258,5 @@
   </visual>
   <collision>
-    <origin xyz="0.252596 -0.314341 -0.447766" rpy="0 0 0"/>
+    <origin xyz="0.252653 -0.314341 -0.453038" rpy="0 0 0"/>
     <geometry>
       <mesh filename="package://ERC22_URDF_description/meshes/Right_leg_double_1.stl" scale="0.001 0.001 0.001"/>
@@ -264,72 +264,72 @@
   </collision>
 </link>
-<joint name="Revoluci�n34" type="continuous">
-  <origin xyz="0.393441 -0.383158 0.365642" rpy="0 0 0"/>
+<joint name="S_LF" type="continuous">
+  <origin xyz="0.391355 -0.383158 0.356565" rpy="0 0 0"/>
   <parent link="base_link"/>
   <child link="WLF_supp_1"/>
-  <axis xyz="-0.022692 -0.0 0.999743"/>
-</joint>
-<joint name="Revoluci�n35" type="continuous">
-  <origin xyz="-0.25259 -0.310658 0.447478" rpy="0 0 0"/>
+  <axis xyz="-5e-06 -0.0 1.0"/>
+</joint>
+<joint name="L_DS" type="continuous">
+  <origin xyz="-0.252653 -0.310658 0.453036" rpy="0 0 0"/>
   <parent link="base_link"/>
   <child link="Left_leg_double_1"/>
   <axis xyz="-0.0 1.0 0.0"/>
 </joint>
-<joint name="Revoluci�n36" type="continuous">
-  <origin xyz="-0.173014 -0.0815 -0.086131" rpy="0 0 0"/>
+<joint name="S_LB" type="continuous">
+  <origin xyz="-0.175276 -0.0815 -0.081429" rpy="0 0 0"/>
   <parent link="Left_leg_double_1"/>
   <child link="WLB_supp_1"/>
-  <axis xyz="0.045096 0.0 -0.998983"/>
-</joint>
-<joint name="Revoluci�n37" type="continuous">
-  <origin xyz="0.007185 0.018483 -0.157836" rpy="0 0 0"/>
+  <axis xyz="0.018114 0.0 -0.999836"/>
+</joint>
+<joint name="W_LB" type="continuous">
+  <origin xyz="0.002922 0.018483 -0.157973" rpy="0 0 0"/>
   <parent link="WLB_supp_1"/>
   <child link="WLB_1"/>
-  <axis xyz="-0.003219 -0.999995 -0.000145"/>
-</joint>
-<joint name="Revoluci�n38" type="continuous">
-  <origin xyz="0.234647 -0.0695 -0.236664" rpy="0 0 0"/>
+  <axis xyz="-0.003222 -0.999995 -5.8e-05"/>
+</joint>
+<joint name="W_LM" type="continuous">
+  <origin xyz="0.228173 -0.0695 -0.242912" rpy="0 0 0"/>
   <parent link="Left_leg_double_1"/>
   <child link="WLM_1"/>
   <axis xyz="-0.0 1.0 0.0"/>
 </joint>
-<joint name="Revoluci�n39" type="continuous">
-  <origin xyz="0.003043 0.018483 -0.139967" rpy="0 0 0"/>
+<joint name="W_LF" type="continuous">
+  <origin xyz="-0.000133 0.018483 -0.14" rpy="0 0 0"/>
   <parent link="WLF_supp_1"/>
   <child link="WLF_1"/>
-  <axis xyz="0.00721 -0.999974 0.000164"/>
-</joint>
-<joint name="Revoluci�n40" type="continuous">
-  <origin xyz="0.393337 0.386841 0.36517" rpy="0 0 0"/>
+  <axis xyz="0.007212 -0.999974 0.0"/>
+</joint>
+<joint name="S_RF" type="continuous">
+  <origin xyz="0.391354 0.386841 0.356561" rpy="0 0 0"/>
   <parent link="base_link"/>
   <child link="WRF_supp_1"/>
-  <axis xyz="0.021515 -0.0 -0.999769"/>
-</joint>
-<joint name="Revoluci�n41" type="continuous">
-  <origin xyz="-0.172942 0.08225 -0.086276" rpy="0 0 0"/>
+  <axis xyz="-3e-06 -0.0 -1.0"/>
+</joint>
+<joint name="S_RB" type="continuous">
+  <origin xyz="-0.175153 0.08225 -0.081692" rpy="0 0 0"/>
   <parent link="Right_leg_double_1"/>
   <child link="WRB_supp_1"/>
-  <axis xyz="-0.045935 0.0 0.998944"/>
-</joint>
-<joint name="Revoluci�n42" type="continuous">
-  <origin xyz="0.002929 -0.011538 -0.13997" rpy="0 0 0"/>
+  <axis xyz="-0.019617 0.0 0.999808"/>
+</joint>
+<joint name="W_RF" type="continuous">
+  <origin xyz="-8.4e-05 -0.011538 -0.14" rpy="0 0 0"/>
   <parent link="WRF_supp_1"/>
   <child link="WRF_1"/>
-  <axis xyz="-0.00721 -0.999974 -0.000155"/>
-</joint>
-<joint name="Revoluci�n43" type="continuous">
-  <origin xyz="0.234845 0.07025 -0.236467" rpy="0 0 0"/>
+  <axis xyz="-0.007212 -0.999974 0.0"/>
+</joint>
+<joint name="W_RM" type="continuous">
+  <origin xyz="0.228538 0.07025 -0.242568" rpy="0 0 0"/>
   <parent link="Right_leg_double_1"/>
   <child link="WRM_1"/>
   <axis xyz="0.0 1.0 -0.0"/>
 </joint>
-<joint name="Revoluci�n44" type="continuous">
-  <origin xyz="0.007258 -0.018484 -0.157833" rpy="0 0 0"/>
+<joint name="W_RB" type="continuous">
+  <origin xyz="0.003099 -0.018484 -0.15797" rpy="0 0 0"/>
   <parent link="WRB_supp_1"/>
   <child link="WRB_1"/>
   <axis xyz="-0.0 -1.0 0.0"/>
 </joint>
-<joint name="Revoluci�n45" type="continuous">
-  <origin xyz="-0.252596 0.314341 0.447766" rpy="0 0 0"/>
+<joint name="R_DS" type="continuous">
+  <origin xyz="-0.252653 0.314341 0.453038" rpy="0 0 0"/>
   <parent link="base_link"/>
   <child link="Right_leg_double_1"/>

Commit message: Controllers, model, and two working cameras

File: urdf/ERC22_URDF.xacro (robot description, xacro)
@@ -264,4 +264,45 @@
   </collision>
 </link>
+  <!-- Camera -->
+<link name="camera_link_left">
+  <collision>
+    <origin xyz="0 0 0" rpy="0 0 0"/>
+    <geometry>
+  <box size="0.05 0.05 0.05"/>
+    </geometry>
+  </collision>
+  <visual>
+    <origin xyz="0 0 0" rpy="0 0 0"/>
+    <geometry>
+  <box size="0.05 0.05 0.05"/>
+    </geometry>
+    <material name="red"/>
+  </visual>
+  <inertial>
+    <mass value="1e-5" />
+    <origin xyz="0 0 0" rpy="0 0 0"/>
+    <inertia ixx="1e-6" ixy="0" ixz="0" iyy="1e-6" iyz="0" izz="1e-6" />
+  </inertial>
+</link>
+<link name="camera_link_right">
+  <collision>
+    <origin xyz="0 0 0" rpy="0 0 0"/>
+    <geometry>
+  <box size="0.05 0.05 0.05"/>
+    </geometry>
+  </collision>
+  <visual>
+    <origin xyz="0 0 0" rpy="0 0 0"/>
+    <geometry>
+  <box size="0.05 0.05 0.05"/>
+    </geometry>
+    <material name="red"/>
+  </visual>
+  <inertial>
+    <mass value="1e-5" />
+    <origin xyz="0 0 0" rpy="0 0 0"/>
+    <inertia ixx="1e-6" ixy="0" ixz="0" iyy="1e-6" iyz="0" izz="1e-6" />
+  </inertial>
+</link>
 <joint name="S_LF" type="continuous">
   <origin xyz="0.391355 -0.383158 0.356565" rpy="0 0 0"/>
@@ -336,3 +377,15 @@
   <axis xyz="0.0 1.0 -0.0"/>
 </joint>
+<joint name="camera_joint_left" type="fixed">
+  <axis xyz="0 1 0" />
+  <origin xyz="0.285 0.23 0.58" rpy="0 0 0.785"/>
+  <parent link="base_link"/>
+  <child link="camera_link_left"/>
+</joint>
+<joint name="camera_joint_right" type="fixed">
+  <axis xyz="0 1 0" />
+  <origin xyz="0.285 -0.23 0.58" rpy="0 0 -0.785"/>
+  <parent link="base_link"/>
+  <child link="camera_link_right"/>
+</joint>
 </robot>

File: urdf/materials.xacro (robot description, xacro)
@@ -4,3 +4,6 @@
   <color rgba="0.700 0.700 0.700 1.000"/>
 </material>
+<material name="red">
+  <color rgba="1.0 0.0 0.0 1.000"/>
+</material>
 </robot>
